File: schematc-io.kicad_sch (KiCad schematic)
At the start: 0 parts

Commit message: Repair & add IO schema
Parts:
- added C27 (x3): 4n7, Capacitor_SMD:C_1206_3216Metric, symbol Device:C
- added C31 (x2): 20n, Capacitor_SMD:C_1206_3216Metric, symbol Device:C
- added C7 (x2): 100n, Capacitor_SMD:C_1206_3216Metric, symbol Device:C
- added D2, D3, D4: LED, Diode_SMD:D_1206_3216Metric, symbol Device:LED
- added D5: SP0502BAJT, Package_TO_SOT_SMD:SOT-323_SC-70, symbol Power_Protection:SP0502BAJT
- added D8 (x2): PMEG10020, symbol Diode:1N5819
- added IC1: AD8544ARUZ-REEL, library:SOP65P640X120-14N, symbol ad8544:AD8544ARUZ-REEL
- added MOSFET1 (x2): PMPB15XP_115, symbol mosfet logic:PMPB15XP_115
- added R14, R15: 1k, Resistor_SMD:R_1206_3216Metric, symbol Device:R
- added R16: 10k, Resistor_SMD:R_1206_3216Metric, symbol Device:R
- added R17: 60, Resistor_SMD:R_1206_3216Metric, symbol Device:R
- added R18 (x2): 180R, LED_SMD:LED_1206_3216Metric, symbol Device:R
- added R18: 60, LED_SMD:LED_1206_3216Metric, symbol Device:R
- added R2, R3, R4: 1k, LED_SMD:LED_1206_3216Metric, symbol Device:R
- added R2: 100R, LED_SMD:LED_1206_3216Metric, symbol Device:R
- added R2 (x3): 10k, LED_SMD:LED_1206_3216Metric, symbol Device:R
- added R24, R25: 100R, Resistor_SMD:R_1206_3216Metric, symbol Device:R
- added R26 (x2): 100R 0,5W, Resistor_SMD:R_2512_6332Metric, symbol Device:R
- added TP1, TP2: GND, symbol Connector:TestPoint
- added TP10: I/O 2, symbol Connector:TestPoint
- added TP11: I/O 3, symbol Connector:TestPoint
- added TP12: I/O 4, symbol Connector:TestPoint
- added TP3, TP4: +12V, symbol Connector:TestPoint
- added TP5, TP6: +5V, symbol Connector:TestPoint
- added TP7, TP8: +3.3V, symbol Connector:TestPoint
- added TP9: I/O 1, symbol Connector:TestPoint
- added U3: SN65HVD232, Package_SO:SOIC-8_3.9x4.9mm_P1.27mm, symbol Interface_CAN_LIN:SN65HVD232
Connections:
- new net: MOSFET1.3, R18.1 (x2)
- new net: R14.1, TP9.1
- new net: D4.1 (K), R4.1
- new net: C27.1, R17.1, R18.1
- new net: R24.1, TP11.1
- new net: D3.1 (K), R2.1
- new net: C31.2, R26.1 (x2)
- new net: R25.1, TP12.1
- new net: IC1.5 (+IN_B), R16.2, R2.1
- new net: D2.1 (K), R3.1
- new net: R15.1, TP10.1
- new net +12V: D8.1 (K), D8.1 (K), TP3.1, TP4.1
- new net +3.3V: C7.1, C7.1, D4.2 (A), IC1.4 (V+), TP7.1, TP8.1, U3.3 (VCC)
- new net +5V: TP5.1, TP6.1
- new net CANH: D5.1 (K), R17.2, U3.7 (CANH)
- new net CANL: D5.2 (K), R18.2, U3.6 (CANL)
- new net CAN_RX: U3.1 (D)
- new net CAN_TX: U3.4 (R)
- new net C_P: IC1.10 (+IN_C), R2.1
- new net C_P_MCU: C27.1, IC1.8 (OUT_C), IC1.9 (-IN_C)
- new net GND: C27.2, C27.2, C27.2, C7.2, C7.2, D5.3 (A), IC1.11 (GND), MOSFET1.4, MOSFET1.4, MOSFET1.8, MOSFET1.8, R2.2, R2.2, R2.2, R2.2, R2.2, R26.2, R26.2, R3.2, R4.2, TP1.1, TP2.1, U3.2 (GND)
- new net I/O_1_MCU: R14.2
- new net I/O_2_MCU: R15.2
- new net I/O_3_MCU: R2.1, R24.2
- new net I/O_4_MCU: R2.1, R25.2
- new net LED_CAN_STATUS: D3.2 (A)
- new net LED_MCU_STATUS: D2.2 (A)
- new net PURGE_VALVE: C31.1, D8.2 (A), MOSFET1.7
- new net PURGE_VALVE_MCU: R18.2
- new net VALVE: C31.1, D8.2 (A), MOSFET1.7
- new net VALVE_MCU: R18.2
- new net V_P: R16.1
- new net V_P_MCU: C27.1, IC1.6 (-IN_B), IC1.7 (OUT_B)
- no-connect marks 0 -> 6
Other:
- note added: "CAN Transceiver"
- note added: "Policzyć dzielnik napięcia z 5V na 3,3V"
- note added: "Purge valve driver"
- note added: "Signal diodes"
- note added: "Termination node (resistors and capacitor) may be omitted during assembly if not required."
- note added: "Test points"
- note added: "Valve driver"
- note added: "Voltage & Current mesurment"
- note added: "Wzmocnienie napięcia z prądu?"
- company: (none) -> Hydrogreen Pollub
- title: (none) -> Fuel Cell Control Unit  (FCCU)
