File: schematc-io.kicad_sch (KiCad schematic)
At the start: 47 parts, among them IC1 AD8544ARUZ-REEL, U3 SN65HVD232

Commit message: Add footprints, Placing MCU
Parts:
- D8: footprint (none) -> Diode_SMD:DIOAD1414W86L464D238
- MOSFET1: footprint (none) -> Transistor_Power_Module:PMPB15XPAX
- R2: value 10k -> 5k
- TP1, TP10, TP11, TP12, TP2, TP3, TP4, TP5, TP6, TP7, TP8, TP9: footprint (none) -> Connector_PinHeader_2.00mm:PinHeader_1x01_P2.00mm_Vertical
Connections:
- net PURGE_VALVE: no longer C31.1, D8.2 (A)
- net VALVE: no longer C31.1, D8.2 (A)
- new net: C31.1, D8.2 (A) (x2)
- no-connect marks 6 -> 14
Other:
- note added: "5V/3 = 1,666...V 1,666V*2 = 3,333...V 15k/3 = 5k 5k*2 = 10k"
- moved on the sheet: C27, C31, C7, D2, D3, D4, D8, MOSFET1, R14, R15, R16, R18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

Commit message: Drawing PCB
Connections:
- net CANH: now also D5.2 (K); no longer D5.1 (K)
- net CANL: now also D5.1 (K); no longer D5.2 (K)
Changed lines of the file:
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@@
   (junction (at 256.54 135.255) (diameter 0) (color 0 0 0 0)
   )
-  (junction (at 132.207 57.912) (diameter 0) (color 0 0 0 0)
+  (junction (at 127.127 57.912) (diameter 0) (color 0 0 0 0)
   )
   (junction (at 33.02 112.395) (diameter 0) (color 0 0 0 0)
@@
   (junction (at 228.6 154.305) (diameter 0) (color 0 0 0 0)
   )
-  (junction (at 127.127 55.372) (diameter 0) (color 0 0 0 0)
+  (junction (at 132.207 55.372) (diameter 0) (color 0 0 0 0)
   )
   (no_connect (at 91.44 118.11))
@@
     (stroke (width 0) (type default))
   )
+  (wire (pts (xy 127.127 57.912) (xy 127.127 65.532))
+    (stroke (width 0) (type default))
+  )
   (wire (pts (xy 76.2 136.525) (xy 91.44 136.525))
     (stroke (width 0) (type default))
@@
     (stroke (width 0) (type default))
   )
-  (wire (pts (xy 132.207 57.912) (xy 139.827 57.912))
+  (wire (pts (xy 119.507 57.912) (xy 127.127 57.912))
     (stroke (width 0) (type default))
   )
@@
     (stroke (width 0) (type default))
   )
-  (wire (pts (xy 109.347 55.372) (xy 127.127 55.372))
+  (wire (pts (xy 109.347 55.372) (xy 132.207 55.372))
     (stroke (width 0) (type default))
   )
@@
     (stroke (width 0) (type default))
   )
-  (wire (pts (xy 127.127 55.372) (xy 139.827 55.372))
-    (stroke (width 0) (type default))
-  )
   (wire (pts (xy 262.89 123.19) (xy 256.54 123.19))
     (stroke (width 0) (type default))
@@
     (stroke (width 0) (type default))
   )
+  (wire (pts (xy 127.127 57.912) (xy 139.827 57.912))
+    (stroke (width 0) (type default))
+  )
   (wire (pts (xy 97.917 57.912) (xy 119.507 57.912))
     (stroke (width 0) (type default))
@@
     (stroke (width 0) (type default))
   )
+  (wire (pts (xy 132.207 55.372) (xy 139.827 55.372))
+    (stroke (width 0) (type default))
+  )
   (wire (pts (xy 199.39 93.345) (xy 240.03 93.345))
     (stroke (width 0) (type default))
@@
     (stroke (width 0) (type default))
   )
+  (wire (pts (xy 132.207 55.372) (xy 132.207 65.532))
+    (stroke (width 0) (type default))
+  )
   (wire (pts (xy 262.255 153.035) (xy 256.54 153.035))
     (stroke (width 0) (type default))
@@
     (stroke (width 0) (type default))
   )
-  (wire (pts (xy 132.207 57.912) (xy 132.207 65.532))
-    (stroke (width 0) (type default))
-  )
   (wire (pts (xy 204.47 39.37) (xy 204.47 47.625))
     (stroke (width 0) (type default))
@@
     (stroke (width 0) (type default))
   )
-  (wire (pts (xy 127.127 55.372) (xy 127.127 65.532))
-    (stroke (width 0) (type default))
-  )
   (wire (pts (xy 77.597 33.782) (xy 77.597 32.512))
     (stroke (width 0) (type default))
@@
     (stroke (width 0) (type default))
   )
-  (wire (pts (xy 119.507 57.912) (xy 132.207 57.912))
-    (stroke (width 0) (type default))
-  )

Commit message: Changing resistance of  Voltage divider
Parts:
- R16: value 10k -> 5k
- R2: value 5k -> 10k
Changed lines of the file:
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@@
       (effects (font (size 1.27 1.27)))
     )
-    (property "Value" "10k" (at 128.905 116.205 90)
+    (property "Value" "5k" (at 128.905 116.205 90)
       (effects (font (size 1.27 1.27)))
     )
@@
       (effects (font (size 1.27 1.27)) (justify left))
     )
-    (property "Value" "5k" (at 124.46 125.095 0)
-      (effects (font (size 1.27 1.27)) (justify left))
-    )
+    (property "Value" "10k" (at 124.46 125.095 0)
+      (effects (font (size 1.27 1.27)) (justify left))
+    )

Commit message: Adding connector for Hydrogen Sensor
Parts:
- added J4: Conn_01x04, Connector_Molex:Molex_KK-396_A-41792-0004_1x04_P3.96mm_Horizontal, symbol Connector_Generic:Conn_01x04
- added R31, R32: 1k, Resistor_SMD:R_1206_3216Metric, symbol Library:R
- R26: renamed from R2; value 100R -> 150R
- renumbered C27 to C26, C27 to C30, C7 to C33, R2 to R17, R2 to R35, R2 to R36
Connections:
- net +5V: now also J4.3 (Pin_3)
- net GND: now also J4.4 (Pin_4); no longer R26.2
- net C_P: no longer names the net of IC1.10 (+IN_C)
- net C_P: now also R26.2; no longer R26.1
- net C_P_MCU renamed PRESSURE_SENSOR_I_MCU
- net PRESSURE_SENSOR_I_MCU: now also R31.1; no longer IC1.9 (-IN_C)
- net V_P renamed PRESSURE_SENSOR_V
- net V_P_MCU renamed PRESSURE_SENSOR_V_MCU
- net PRESSURE_SENSOR_V_MCU: now also R32.2; no longer IC1.6 (-IN_B)
- new net: IC1.6 (-IN_B), R32.1
- new net: IC1.9 (-IN_C), R31.2
- new net HYDROGEN_SENSOR_: J4.2 (Pin_2)
- new net HYDROGEN_SENSOR_ADC: J4.1 (Pin_1)
- new net PRESSURE_SENSOR_I: R26.1
Other:
- note added: "HYDROGEN SENSOR"
- moved on the sheet: C26, C30, C33, R16, R17, R26

Commit message: Adding motor driver unit
Parts:
- D8: footprint Diode_SMD:DIOAD1414W86L464D238 -> Diode_SMD:PMEG10020ELR
- R18, R2, R26, R3, R4: footprint LED_SMD:LED_1206_3216Metric -> Resistor_SMD:R_1206_3216Metric
Connections:
- net HYDROGEN_SENSOR_: now also J4.1 (Pin_1); no longer J4.2 (Pin_2)
- net HYDROGEN_SENSOR_ADC: now also J4.2 (Pin_2); no longer J4.1 (Pin_1)
- net PURGE_VALVE: now also MOSFET1.1, MOSFET1.2, MOSFET1.5, MOSFET1.6
- net VALVE: now also MOSFET1.1, MOSFET1.2, MOSFET1.5, MOSFET1.6
Other:
- note removed: "Wzmocnienie napięcia z prądu?"
- moved on the sheet: C26, C27, C30, C31, C33, C7, D2, D3, D4, D5, D8, IC1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

Commit message: Change of dimensions
Connections:
- net PURGE_VALVE: now also C31.1, D8.2 (A)
- net VALVE: now also C31.1, D8.2 (A)
- no-connect marks 14 -> 10
Other:
- moved on the sheet: C31, D8, R26
Changed lines of the file:
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@@
 	)
 	(junction
+		(at 266.7 31.75)
+		(diameter 0)
+		(color 0 0 0 0)
+	)
+	(junction
 		(at 115.57 55.88)
 		(diameter 0)
@@
 	)
 	(junction
+		(at 254 77.47)
+		(diameter 0)
+		(color 0 0 0 0)
+	)
+	(junction
 		(at 262.255 152.4)
 		(diameter 0)
@@
 	)
 	(no_connect
-		(at 251.46 34.29)
-	)
-	(no_connect
 		(at 57.15 107.95)
 	)
@@
 	)
 	(no_connect
-		(at 246.38 80.01)
-	)
-	(no_connect
 		(at 57.15 105.41)
 	)
 	(no_connect
-		(at 251.46 36.83)
-	)
-	(no_connect
 		(at 57.15 110.49)
 	)
 	(no_connect
-		(at 246.38 82.55)
-	)
-	(no_connect
 		(at 205.74 77.47)
 	)
@@
 	(wire
 		(pts
-			(xy 266.065 28.575) (xy 266.065 31.75)
+			(xy 266.7 29.21) (xy 266.7 31.75)
 		)
 		(stroke
@@
 	(wire
 		(pts
+			(xy 254 77.47) (xy 260.35 77.47)
+		)
+		(stroke
+			(width 0)
+			(type default)
+		)
+	)
+	(wire
+		(pts
 			(xy 251.46 34.29) (xy 254 34.29)
 		)
@@
 	(wire
 		(pts
-			(xy 248.92 77.47) (xy 260.35 77.47)
+			(xy 248.92 77.47) (xy 254 77.47)
 		)
 		(stroke
@@
 	(wire
 		(pts
-			(xy 266.065 46.99) (xy 266.065 47.625)
+			(xy 266.7 46.99) (xy 266.7 47.625)
 		)
 		(stroke
@@
 	(wire
 		(pts
-			(xy 251.46 47.625) (xy 266.065 47.625)
+			(xy 266.7 31.75) (xy 272.288 31.75)
+		)
+		(stroke
+			(width 0)
+			(type default)
+		)
+	)
+	(wire
+		(pts
+			(xy 251.46 47.625) (xy 266.7 47.625)
 		)
 		(stroke
@@
 	(wire
 		(pts
-			(xy 254 31.75) (xy 272.288 31.75)
+			(xy 254 31.75) (xy 266.7 31.75)
 		)
 		(stroke
@@
 	(symbol
 		(lib_id "power:+12V")
-		(at 266.065 20.955 0)
+		(at 266.7 21.59 0)
 		(unit 1)
 		(exclude_from_sim no)
@@
 		(fields_autoplaced yes)
 		(property "Reference" "#PWR040"
-			(at 266.065 24.765 0)
+			(at 266.7 25.4 0)
 			(effects
 				(font
@@
 		)
 		(property "Value" "+12V"
-			(at 266.065 15.875 0)
+			(at 266.7 16.51 0)
 			(effects
 				(font
@@
 		)
 		(property "Footprint" ""
-			(at 266.065 20.955 0)
+			(at 266.7 21.59 0)
 			(effects
 				(font
@@
 		)
 		(property "Datasheet" ""
-			(at 266.065 20.955 0)
+			(at 266.7 21.59 0)
 			(effects
 				(font
@@
 		)
 		(property "Description" ""
-			(at 266.065 20.955 0)
+			(at 266.7 21.59 0)
 			(effects
 				(font
@@
 	(symbol
 		(lib_id "Device:R")
-		(at 266.065 43.18 0)
+		(at 266.7 43.18 0)
 		(unit 1)
 		(exclude_from_sim no)
@@
 		(fields_autoplaced yes)
 		(property "Reference" "R26"
-			(at 268.605 41.91 0)
+			(at 269.24 41.91 0)
 			(effects
 				(font
@@
 		)
 		(property "Value" "100R 0,5W"
-			(at 268.605 44.45 0)
+			(at 269.24 44.45 0)
 			(effects
 				(font
@@
 		)
 		(property "Footprint" "Resistor_SMD:R_2512_6332Metric"
-			(at 264.287 43.18 90)
+			(at 264.922 43.18 90)
 			(effects
 				(font
@@
 		)
 		(property "Datasheet" "~"
-			(at 266.065 43.18 0)
+			(at 266.7 43.18 0)
 			(effects
 				(font
@@
 		)
 		(property "Description" ""
-			(at 266.065 43.18 0)
+			(at 266.7 43.18 0)
 			(effects
 				(font
@@
 	(symbol
 		(lib_id "Diode:1N5819")
-		(at 266.065 24.765 270)
+		(at 266.7 25.4 270)
 		(unit 1)
 		(exclude_from_sim no)
@@
 		(fields_autoplaced yes)
 		(property "Reference" "D8"
-			(at 268.605 23.1775 90)
+			(at 269.24 23.8125 90)
 			(effects
 				(font
@@
 		)
 		(property "Value" "PMEG10020"
-			(at 268.605 25.7175 90)
+			(at 269.24 26.3525 90)
 			(effects
 				(font
@@
 		)
 		(property "Footprint" "Diode_SMD:PMEG10020ELR"
-			(at 261.62 24.765 0)
+			(at 262.255 25.4 0)
 			(effects
 				(font
@@
 		)
 		(property "Datasheet" "http://www.vishay.com/docs/88525/1n5817.pdf"
-			(at 266.065 24.765 0)
+			(at 266.7 25.4 0)
 			(effects
 				(font
@@
 		)
 		(property "Description" ""
-			(at 266.065 24.765 0)
+			(at 266.7 25.4 0)
 			(effects
 				(font
@@
 	(symbol
 		(lib_id "Device:C")
-		(at 266.065 35.56 0)
+		(at 266.7 35.56 0)
 		(unit 1)
 		(exclude_from_sim no)
@@
 		(dnp no)
 		(property "Reference" "C31"
-			(at 269.875 35.56 0)
+			(at 270.51 35.56 0)
 			(effects
 				(font
@@
 		)
 		(property "Value" "20n"
-			(at 269.875 38.1 0)
+			(at 270.51 38.1 0)
 			(effects
 				(font
@@
 		)
 		(property "Footprint" "Capacitor_SMD:C_1206_3216Metric"
-			(at 267.0302 39.37 0)
+			(at 267.6652 39.37 0)
 			(effects
 				(font
@@
 		)
 		(property "Datasheet" "~"
-			(at 266.065 35.56 0)
+			(at 266.7 35.56 0)
 			(effects
 				(font
@@
 		)
 		(property "Description" ""
-			(at 266.065 35.56 0)
+			(at 266.7 35.56 0)
 			(effects
 				(font

Commit message: Change of PRESSURE_SENSOR_I circuit
Parts:
- added R38: 0, Resistor_SMD:R_1206_3216Metric, symbol Library:R
Connections:
- net GND: now also R26.1
- net PRESSURE_SENSOR_I: now also R26.2, R38.1; no longer R26.1
- net at IC1.10 (+IN_C): now also R38.2; no longer R26.2
Other:
- moved on the sheet: R26
Changed lines of the file:
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@@
 	)
 	(junction
+		(at 46.99 107.95)
+		(diameter 0)
+		(color 0 0 0 0)
+	)
+	(junction
 		(at 262.255 152.4)
 		(diameter 0)
@@
 	(wire
 		(pts
+			(xy 46.99 107.95) (xy 48.26 107.95)
+		)
+		(stroke
+			(width 0)
+			(type default)
+		)
+	)
+	(wire
+		(pts
 			(xy 103.505 120.65) (xy 97.79 120.65)
 		)
@@
 	(wire
 		(pts
+			(xy 46.99 99.06) (xy 46.99 107.95)
+		)
+		(stroke
+			(width 0)
+			(type default)
+		)
+	)
+	(wire
+		(pts
 			(xy 23.749 45.72) (xy 21.209 45.72)
 		)
@@
 	(wire
 		(pts
+			(xy 36.83 107.95) (xy 36.83 114.3)
+		)
+		(stroke
+			(width 0)
+			(type default)
+		)
+	)
+	(wire
+		(pts
 			(xy 254 77.47) (xy 260.35 77.47)
 		)
@@
 	(wire
 		(pts
-			(xy 52.07 109.22) (xy 55.88 109.22)
+			(xy 45.72 107.95) (xy 46.99 107.95)
 		)
 		(stroke
@@
 	(wire
 		(pts
-			(xy 55.88 109.22) (xy 55.88 115.57)
+			(xy 55.88 107.95) (xy 55.88 115.57)
+		)
+		(stroke
+			(width 0)
+			(type default)
+		)
+	)
+	(wire
+		(pts
+			(xy 36.83 107.95) (xy 38.1 107.95)
 		)
 		(stroke
@@
 	(wire
 		(pts
+			(xy 39.37 99.06) (xy 46.99 99.06)
+		)
+		(stroke
+			(width 0)
+			(type default)
+		)
+	)
+	(wire
+		(pts
 			(xy 266.7 31.75) (xy 272.288 31.75)
 		)
@@
 	(hierarchical_label "PRESSURE_SENSOR_I"
 		(shape input)
-		(at 44.45 109.22 180)
+		(at 39.37 99.06 180)
 		(fields_autoplaced yes)
 		(effects
@@
 	(symbol
 		(lib_id "Device:R")
-		(at 48.26 109.22 90)
+		(at 41.91 107.95 90)
 		(unit 1)
 		(exclude_from_sim no)
@@
 		(dnp no)
 		(property "Reference" "R26"
-			(at 50.038 104.648 90)
+			(at 43.688 103.378 90)
 			(effects
 				(font
@@
 		)
 		(property "Value" "150R"
-			(at 50.8 106.934 90)
+			(at 44.45 105.664 90)
 			(effects
 				(font
@@
 		)
 		(property "Footprint" "Resistor_SMD:R_1206_3216Metric"
-			(at 48.26 110.998 90)
+			(at 41.91 109.728 90)
 			(effects
 				(font
@@
 		)
 		(property "Datasheet" "~"
-			(at 48.26 109.22 0)
+			(at 41.91 107.95 0)
 			(effects
 				(font
@@
 		)
 		(property "Description" ""
-			(at 48.26 109.22 0)
+			(at 41.91 107.95 0)
 			(effects
 				(font
@@
 	)
 	(symbol
+		(lib_name "GND_2")
+		(lib_id "power:GND")
+		(at 36.83 114.3 0)
+		(unit 1)
+		(exclude_from_sim no)
+		(in_bom yes)
+		(on_board yes)
+		(dnp no)
+		(fields_autoplaced yes)
+		(property "Reference" "#PWR079"
+			(at 36.83 120.65 0)
+			(effects
+				(font
+					(size 1.27 1.27)
+				)
+				(hide yes)
+			)
+		)
+		(property "Value" "GND"
+			(at 36.83 119.38 0)
+			(effects
+				(font
+					(size 1.27 1.27)
+				)
+				(hide yes)
+			)
+		)
+		(property "Footprint" ""
+			(at 36.83 114.3 0)
+			(effects
+				(font
+					(size 1.27 1.27)
+				)
+				(hide yes)
+			)
+		)
+		(property "Datasheet" ""
+			(at 36.83 114.3 0)
+			(effects
+				(font
+					(size 1.27 1.27)
+				)
+				(hide yes)
+			)
+		)
+		(property "Description" "Power symbol creates a global label with name \"GND\" , ground"
+			(at 36.83 114.3 0)
+			(effects
+				(font
+					(size 1.27 1.27)
+				)
+				(hide yes)
+			)
+		)
+		(pin "1"
+		)
+		(instances
+			(project "schematic-main"
+				(path "/c9ad7189-d3b2-414a-9743-efd8e57cd755/e4695f4d-6fa6-4597-a598-6a2f28a255eb"
+					(reference "#PWR079")
+					(unit 1)
+				)
+			)
+		)
+	)
+	(symbol
 		(lib_id "power:GND")
 		(at 125.73 73.66 0)
@@
 					(unit 1)
 				)
+			)
+		)
+	)
+	(symbol
+		(lib_id "Library:R")
+		(at 52.07 107.95 90)
+		(unit 1)
+		(exclude_from_sim no)
+		(in_bom yes)
+		(on_board yes)
+		(dnp no)
+		(fields_autoplaced yes)
+		(property "Reference" "R38"
+			(at 52.07 101.6 90)
+			(effects
+				(font
+					(size 1.27 1.27)
+				)
+			)
+		)
+		(property "Value" "0"
+			(at 52.07 104.14 90)
+			(effects
+				(font
+					(size 1.27 1.27)
+				)
+			)
+		)
+		(property "Footprint" "Resistor_SMD:R_1206_3216Metric"
+			(at 52.07 109.728 90)
+			(effects
+				(font
+					(size 1.27 1.27)
+				)
+				(hide yes)
+			)
+		)
+		(property "Datasheet" "~"
+			(at 52.07 107.95 0)
+			(effects
+				(font
+					(size 1.27 1.27)
+				)
+				(hide yes)
+			)
+		)
+		(property "Description" "Resistor"
+			(at 52.07 107.95 0)
+			(effects
+				(font
+					(size 1.27 1.27)
+				)
+				(hide yes)
+			)
+		)
+		(pin "1"
+		)
+		(pin "2"
+		)
+		(instances
+			(project "schematic-main"
+				(path "/c9ad7189-d3b2-414a-9743-efd8e57cd755/e4695f4d-6fa6-4597-a598-6a2f28a255eb"
+					(reference "R38")
+					(unit 1)
+				)

Commit message: Change of socket for Hudrogen sensor
Parts:
- J4: footprint Connector_Molex:Molex_KK-396_A-41792-0004_1x04_P3.96mm_Horizontal -> Lib:39-30-104Y
Connections:
- net +5V: now also J4.1 (Pin_1); no longer J4.3 (Pin_3)
- net GND: now also J4.2 (Pin_2); no longer J4.4 (Pin_4)
- net HYDROGEN_SENSOR_: now also J4.3 (Pin_3); no longer J4.1 (Pin_1)
- net HYDROGEN_SENSOR_ADC: now also J4.4 (Pin_4); no longer J4.2 (Pin_2)
- no-connect marks 10 -> 6
Changed lines of the file:
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@@
 	)
 	(no_connect
-		(at 210.82 34.29)
-	)
-	(no_connect
 		(at 57.15 105.41)
 	)
@@
 		(at 57.15 110.49)
 	)
-	(no_connect
-		(at 205.74 77.47)
-	)
-	(no_connect
-		(at 210.82 31.75)
-	)
-	(no_connect
-		(at 205.74 80.01)
-	)
 	(wire
 		(pts
@@
 	(wire
 		(pts
+			(xy 102.87 156.21) (xy 102.87 157.48)
+		)
+		(stroke
+			(width 0)
+			(type default)
+		)
+	)
+	(wire
+		(pts
 			(xy 26.797 40.386) (xy 26.797 45.72)
 		)
@@
 	(wire
 		(pts
-			(xy 102.87 165.1) (xy 102.87 162.56)
+			(xy 105.41 53.34) (xy 128.27 53.34)
 		)
 		(stroke
@@
 	(wire
 		(pts
-			(xy 105.41 53.34) (xy 128.27 53.34)
+			(xy 266.7 29.21) (xy 266.7 31.75)
 		)
 		(stroke
@@
 	(wire
 		(pts
-			(xy 266.7 29.21) (xy 266.7 31.75)
+			(xy 248.92 63.5) (xy 248.92 66.04)
 		)
 		(stroke
@@
 	(wire
 		(pts
-			(xy 248.92 63.5) (xy 248.92 66.04)
+			(xy 254 92.71) (xy 254 93.345)
 		)
 		(stroke
@@
 	(wire
 		(pts
-			(xy 254 92.71) (xy 254 93.345)
+			(xy 100.33 154.94) (xy 102.87 154.94)
 		)
 		(stroke
@@
 	(wire
 		(pts
+			(xy 100.33 156.21) (xy 102.87 156.21)
+		)
+		(stroke
+			(width 0)
+			(type default)
+		)
+	)
+	(wire
+		(pts
 			(xy 234.315 153.67) (xy 234.315 160.02)
 		)
@@
 	(hierarchical_label "HYDROGEN_SENSOR_ADC"
 		(shape output)
-		(at 102.87 157.48 180)
+		(at 102.87 162.56 180)
 		(fields_autoplaced yes)
 		(effects
@@
 	(hierarchical_label "HYDROGEN_SENSOR_"
 		(shape output)
-		(at 102.87 154.94 180)
+		(at 102.87 160.02 180)
 		(fields_autoplaced yes)
 		(effects
@@
 			)
 		)
-		(property "Footprint" "Connector_Molex:Molex_KK-396_A-41792-0004_1x04_P3.96mm_Horizontal"
+		(property "Footprint" "Lib:39-30-104Y"
 			(at 107.95 157.48 0)
 			(effects
@@
 		(lib_name "GND_1")
 		(lib_id "power:GND")
-		(at 102.87 165.1 0)
+		(at 100.33 156.21 0)
 		(unit 1)
 		(exclude_from_sim no)
@@
 		(fields_autoplaced yes)
 		(property "Reference" "#PWR040"
-			(at 102.87 171.45 0)
+			(at 100.33 162.56 0)
 			(effects
 				(font
@@
 		)
 		(property "Value" "GND"
-			(at 102.87 170.18 0)
+			(at 100.33 161.29 0)
 			(effects
 				(font
@@
 		)
 		(property "Footprint" ""
-			(at 102.87 165.1 0)
+			(at 100.33 156.21 0)
 			(effects
 				(font
@@
 		)
 		(property "Datasheet" ""
-			(at 102.87 165.1 0)
+			(at 100.33 156.21 0)
 			(effects
 				(font
@@
 		)
 		(property "Description" "Power symbol creates a global label with name \"GND\" , ground"
-			(at 102.87 165.1 0)
+			(at 100.33 156.21 0)
 			(effects
 				(font
@@
 		(lib_name "+5V_1")
 		(lib_id "power:+5V")
-		(at 102.87 160.02 90)
+		(at 100.33 154.94 0)
 		(unit 1)
 		(exclude_from_sim no)
@@
 		(on_board yes)
 		(dnp no)
-		(fields_autoplaced yes)
 		(property "Reference" "#PWR071"
-			(at 106.68 160.02 0)
+			(at 100.33 158.75 0)
 			(effects
 				(font
@@
 		)
 		(property "Value" "+5V"
-			(at 99.06 160.0199 90)
+			(at 97.282 153.162 0)
 			(effects
 				(font
 					(size 1.27 1.27)
 				)
-				(justify left)
 			)
 		)
 		(property "Footprint" ""
-			(at 102.87 160.02 0)
+			(at 100.33 154.94 0)
 			(effects
 				(font
@@
 		)
 		(property "Datasheet" ""
-			(at 102.87 160.02 0)
+			(at 100.33 154.94 0)
 			(effects
 				(font
@@
 		)
 		(property "Description" "Power symbol creates a global label with name \"+5V\""
-			(at 102.87 160.02 0)
+			(at 100.33 154.94 0)
 			(effects
 				(font
