File: schematic-main_HCU.kicad_pcb (KiCad board)
At the start: 2 copper layers, 100 x 99.9 mm, 124 parts, among them IC1 AD8544ARUZ-REEL, IC2 LM76202QPWPRQ1, J1 Battery, J10 Motor, J2 CAN, J3 V_P, J4 Conn_01x04, J7 C_P, J8 VALVE, J9 PURGE_VALVE, P1 USB_C_Plug_USB2.0, U2 TPS62933, U3 USBLC6-2P6, U4 ESP32-S3FN8, U5 SN65HVD232, U6 DRV8801PWP, Y1 Crystal_GND24

Commit message: DRC test copmlate
Parts:
- removed J7: C_P, Connector_Molex:39-30-102Y
- J10: value Motor -> Battery
- J3: footprint Connector_Molex:39-30-102Y -> Lib:39-30-104Y
- moved J3 21.4 mm to (114.9, 137.9)
- moved J1 17.2 mm to (63.3, 78.8)
- moved J10 17.2 mm to (63.3, 86.6)
- moved D7 11.1 mm to (74.5, 121.5)
- moved J9 10.8 mm to (63.0, 133.3)
- moved R26 10.8 mm to (112.9, 129.0), turned to 0 degrees
- moved J8 10.7 mm to (62.9, 123.2)
- moved D8 10.6 mm to (73.7, 129.7)
- moved J4 9.40 mm to (135.0, 115.1)
- moved TP1 8.36 mm to (137.4, 139.3)
- moved TP2 8.36 mm to (137.4, 144.3)
- moved C7 5.40 mm to (77.8, 90.0)
- moved D3 5.13 mm to (128.9, 106.2)
- moved C24 4.44 mm to (127.8, 102.2), turned to 90 degrees
- moved R31 4.22 mm to (117.1, 127.4)
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Connections:
- J3 pad 1: /IO/PRESSURE_SENSOR_V -> GND
- J3 pad 2: +12V -> /IO/PRESSURE_SENSOR_V
- P1 pad MH1: (no net) -> GND
- P1 pad MH2: (no net) -> GND
- P1 pad MH3: (no net) -> GND
Routing:
- net GND: track 568.4 -> 497.7 mm, vias 59 -> 106
- net +5V: track 77.4 -> 137.3 mm
- net /VBUS: track 84.2 -> 103.5 mm, vias 2 -> 4
- net /IO/PRESSURE_SENSOR_V: track 13.1 -> 31.5 mm
- net /Power /Vin: track 65.1 -> 79.9 mm
- net +3.3V: track 296.7 -> 310.3 mm, vias 18 -> 15
- net /IO_2/+MOTOR: track 23.6 -> 35.7 mm, vias 0 -> 1
- net /HYDROGEN_SENSOR_ADC: track 49.7 -> 37.7 mm
- net Net-(U2-VIN): track 17.2 -> 27.2 mm
- net /HYDROGEN_SENSOR_: track 32.7 -> 24.2 mm
- net Net-(IC1-+IN_C): track 2.72 -> 9.42 mm
- net /IO_2/-MOTOR: track 13.1 -> 19.2 mm
- net Net-(IC1--IN_C): track 2.88 -> 7.41 mm
- net /IO/CANH: track 28.3 -> 25.0 mm
- net Net-(U2-SW): track 6.82 -> 9.72 mm
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Other:
- board text added: "+M"
- board text added: "-M"
- board text added: "CAN: H L GND"
- board text added: "H2_SENSOR"
- board text added: "HYDROGEN_SENSOR: Bin_s Analog_s GND +5V"
- board text added: "MAIN VALVE GND"
- board text added: "MAIN_VALVE"
- board text added: "Motor"
- board text added: "PRESSURE_SENSOR_I 4-20mA"
- board text added: "PRESSURE_SENSOR_V 5V"
- board text added: "PRESURE_SENSOR"
- board text added: "PURGE VALVE GND"
- board text added: "P_SEN_I"
- board text added: "P_SEN_V"
- board text added: "P_VALVE"
- board text added: "TEST"
- board text removed: "HYDROGEN SENSOR"
- board text removed: "MCU_TEST"
- board text removed: "MOTOR_DRIVER"
- board text removed: "POWER"
- board text removed: "PRESSURE_SENSOR_I"
- board text removed: "PRESSURE_SENSOR_V"
